Commit message: Messing with namespaces
--HG--
branch : namespaces_for_rviz

File: x1_description/urdf/decorations.urdf.xacro (robot description, xacro)
@@ -22,5 +22,5 @@
 -->
 <robot name="x1_decorations" xmlns:xacro="http://ros.org/wiki/xacro">
-  <xacro:macro name="x1_decorate">
+  <xacro:macro name="x1_decorate" params="robot_namespace">
     <!-- Spawn X1 chassis -->
     <link name="top_chassis_link">
@@ -28,5 +28,5 @@
     <!-- Attach chassis to the robot -->
     <joint name="top_chassis_joint" type="fixed">
-      <parent link="base_link" />
+      <parent link="${robot_namespace}/base_link" />
       <child link="top_chassis_link" />
     </joint>
@@ -53,5 +53,5 @@
     <!-- Attach top plate -->
     <joint name="top_plate_joint" type="fixed">
-      <parent link="base_link" />
+      <parent link="${robot_namespace}/base_link" />
       <child link="top_plate_link"/>
       <origin xyz="0.0812 0 0.245" rpy="0 0 0"/>

File: x1_description/urdf/headlight.urdf.xacro (robot description, xacro)
@@ -1,5 +1,5 @@
 <?xml version="1.0"?>
 <robot xmlns:xacro="http://ros.org/wiki/xacro" name="headlight">
-  <xacro:macro name="headlight" params="headlight_prefix xyz rpy">
+  <xacro:macro name="headlight" params="headlight_prefix xyz rpy robot_namespace">
     <link name="${headlight_prefix}_headlight_link">
       <visual>
@@ -20,5 +20,5 @@
     </link>
     <joint name="${headlight_prefix}_headlight" type="fixed">
-      <parent link="base_link"/>
+      <parent link="${robot_namespace}/base_link"/>
       <child link="${headlight_prefix}_headlight_link"/>
       <origin xyz="${xyz}" rpy="${rpy}"/>
@@ -90,5 +90,5 @@
     <gazebo>
       <joint name="${headlight_prefix}_headlight" type="fixed">
-        <parent>base_link</parent>
+        <parent>${robot_namespace}/base_link</parent>
         <child>${headlight_prefix}_headlight::body</child>
       </joint>

File: x1_description/urdf/led.urdf.xacro (robot description, xacro)
@@ -1,5 +1,5 @@
 <?xml version="1.0"?>
 <robot xmlns:xacro="http://ros.org/wiki/xacro" name="led">
-  <xacro:macro name="led" params="led_prefix xyz rpy **plugin_params">
+  <xacro:macro name="led" params="led_prefix xyz rpy **plugin_params robot_namespace">
     <link name="${led_prefix}_led_link">
       <visual name="marker">
@@ -20,5 +20,5 @@
     </link>
     <joint name="${led_prefix}_led" type="fixed">
-      <parent link="base_link"/>
+      <parent link="${robot_namespace}/base_link"/>
       <child link="${led_prefix}_led_link"/>
       <origin xyz="${xyz}" rpy="${rpy}"/>
@@ -85,5 +85,5 @@
     <gazebo>
       <joint name="${led_prefix}_led" type="fixed">
-        <parent>base_link</parent>
+        <parent>${robot_namespace}/base_link</parent>
         <child>${led_prefix}_led::body</child>
       </joint>

File: x1_description/urdf/wheel.urdf.xacro (robot description, xacro)
@@ -22,5 +22,5 @@
 -->
 <robot xmlns:xacro="http://ros.org/wiki/xacro" name="x1_wheel">
-	<xacro:macro name="x1_wheel" params="wheel_prefix *joint_pose">
+	<xacro:macro name="x1_wheel" params="wheel_prefix *joint_pose robot_namespace">
 		<link name="${wheel_prefix}_wheel_link">
 			<inertial>
@@ -50,5 +50,5 @@
 		</gazebo>
 		<joint name="${wheel_prefix}_wheel" type="continuous">
-			<parent link="base_link"/>
+      <parent link="${robot_namespace}/base_link"/>
 			<child link="${wheel_prefix}_wheel_link"/>
 			<xacro:insert_block name="joint_pose"/>

File: x1_description/urdf/x1.urdf.xacro (robot description, xacro)
@@ -53,5 +53,5 @@
   <xacro:property name="wheel_radius" value="0.1651" />
   <!-- Base link is the center of the robot's bottom plate -->
-  <link name="base_link">
+  <link name="$(arg robot_namespace)/base_link">
     <visual>
       <origin xyz="0 0 0" rpy="0 0 3.1416" />
@@ -77,5 +77,5 @@
   <joint name="base_footprint_joint" type="fixed">
     <origin xyz="0 0 ${wheel_vertical_offset - wheel_radius}" rpy="0 0 0" />
-    <parent link="base_link" />
+    <parent link="$(arg robot_namespace)/base_link" />
     <child link="base_footprint" />
   </joint>
@@ -90,5 +90,5 @@
   <joint name="inertial_joint" type="fixed">
     <origin xyz="0 0 0" rpy="0 0 0" />
-    <parent link="base_link" />
+    <parent link="$(arg robot_namespace)/base_link" />
     <child link="inertial_link" />
   </joint>
@@ -98,5 +98,5 @@
   <joint name="imu_joint" type="fixed">
     <origin xyz="$(optenv X1_IMU_XYZ 0.19 0 0.149)" rpy="$(optenv X1_IMU_RPY 0 -1.5708 3.1416)" />
-    <parent link="base_link" />
+    <parent link="$(arg robot_namespace)/base_link" />
     <child link="imu_link" />
   </joint>
@@ -104,37 +104,37 @@
   </gazebo>
   <!-- X1 wheel macros -->
-  <xacro:x1_wheel wheel_prefix="front_left">
+  <xacro:x1_wheel wheel_prefix="front_left" robot_namespace="$(arg robot_namespace)">
     <origin xyz="${wheelbase/2} ${track/2} ${wheel_vertical_offset}" rpy="0 0 0" />
   </xacro:x1_wheel>
-  <xacro:x1_wheel wheel_prefix="front_right">
+  <xacro:x1_wheel wheel_prefix="front_right" robot_namespace="$(arg robot_namespace)">
     <origin xyz="${wheelbase/2} ${-track/2} ${wheel_vertical_offset}" rpy="0 0 0" />
   </xacro:x1_wheel>
-  <xacro:x1_wheel wheel_prefix="rear_left">
+  <xacro:x1_wheel wheel_prefix="rear_left" robot_namespace="$(arg robot_namespace)">
     <origin xyz="${-wheelbase/2} ${track/2} ${wheel_vertical_offset}" rpy="0 0 0" />
   </xacro:x1_wheel>
-  <xacro:x1_wheel wheel_prefix="rear_right">
+  <xacro:x1_wheel wheel_prefix="rear_right" robot_namespace="$(arg robot_namespace)">
     <origin xyz="${-wheelbase/2} ${-track/2} ${wheel_vertical_offset}" rpy="0 0 0" />
   </xacro:x1_wheel>
-  <xacro:x1_decorate />
+  <xacro:x1_decorate robot_namespace="$(arg robot_namespace)"/>
   <!-- Head lights -->
   <xacro:headlight headlight_prefix="left"
-    xyz="0.461459  0.216803 0.124431" rpy="0 0 3.1416" />
+    xyz="0.461459  0.216803 0.124431" rpy="0 0 3.1416" robot_namespace="$(arg robot_namespace)" />
   <xacro:headlight headlight_prefix="center_left"
-    xyz="0.485766 0.0844 0.124431" rpy="0 0 3.1416" />
+    xyz="0.485766 0.0844 0.124431" rpy="0 0 3.1416" robot_namespace="$(arg robot_namespace)" />
   <xacro:headlight headlight_prefix="center_right"
-    xyz="0.485766 -0.0844 0.124431" rpy="0 0 3.1416" />
+    xyz="0.485766 -0.0844 0.124431" rpy="0 0 3.1416" robot_namespace="$(arg robot_namespace)" />
   <xacro:headlight headlight_prefix="right"
-    xyz="0.461459  -0.216803 0.124431" rpy="0 0 3.1416" />
+    xyz="0.461459  -0.216803 0.124431" rpy="0 0 3.1416" robot_namespace="$(arg robot_namespace)" />
    <!-- LEDs -->
-  <xacro:led led_prefix="rear_right" xyz="-0.42493 -0.13619 0.209188" rpy="0 1.573 3.1416">
-    <plugin_params>
-      <block>
-        <duration>0.3</duration>
-        <interval>0.3</interval>
-        <color>1 0.8</color>
-      </block>
-    </plugin_params>
-  </xacro:led>
-  <xacro:led led_prefix="rear_center" xyz="-0.42493 0 0.209188" rpy="0 1.573 3.1416">
+  <xacro:led led_prefix="rear_right" xyz="-0.42493 -0.13619 0.209188" rpy="0 1.573 3.1416" robot_namespace="$(arg robot_namespace)">
+    <plugin_params>
+      <block>
+        <duration>0.3</duration>
+        <interval>0.3</interval>
+        <color>1 0.8</color>
+      </block>
+    </plugin_params>
+  </xacro:led>
+  <xacro:led led_prefix="rear_center" xyz="-0.42493 0 0.209188" rpy="0 1.573 3.1416" robot_namespace="$(arg robot_namespace)">
     <plugin_params>
       <block>
@@ -155,41 +155,41 @@
     </plugin_params>
   </xacro:led>
-  <xacro:led led_prefix="rear_left" xyz="-0.42493 0.13619 0.209188" rpy="0 1.573 3.1416">
-    <plugin_params>
-      <block>
-        <duration>0.3</duration>
-        <interval>0.3</interval>
-        <color>1 0.8</color>
-      </block>
-    </plugin_params>
-  </xacro:led>
-  <xacro:led led_prefix="right_lateral_front" xyz="0.066047 -0.212211 0.209188" rpy="0 1.573 -1.539">
-    <plugin_params>
-      <block>
-        <duration>0.3</duration>
-        <interval>0.3</interval>
-        <color>1 0.8</color>
-      </block>
-    </plugin_params>
-  </xacro:led>
-  <xacro:led led_prefix="right_lateral_rear" xyz="-0.066047 -0.212211 0.209188" rpy="0 1.573 -1.539">
-    <plugin_params>
-      <block>
-        <duration>0.3</duration>
-        <interval>0.3</interval>
-        <color>1 0.8</color>
-      </block>
-    </plugin_params>
-  </xacro:led>
-  <xacro:led led_prefix="left_lateral_front" xyz="0.066047 0.212211 0.209188" rpy="0 1.573 1.539">
-    <plugin_params>
-      <block>
-        <duration>0.3</duration>
-        <interval>0.3</interval>
-        <color>1 0.8</color>
-      </block>
-    </plugin_params>
-  </xacro:led>
-  <xacro:led led_prefix="left_lateral_rear" xyz="-0.066047 0.212211 0.209188" rpy="0 1.573 1.539">
+  <xacro:led led_prefix="rear_left" xyz="-0.42493 0.13619 0.209188" rpy="0 1.573 3.1416" robot_namespace="$(arg robot_namespace)">
+    <plugin_params>
+      <block>
+        <duration>0.3</duration>
+        <interval>0.3</interval>
+        <color>1 0.8</color>
+      </block>
+    </plugin_params>
+  </xacro:led>
+  <xacro:led led_prefix="right_lateral_front" xyz="0.066047 -0.212211 0.209188" rpy="0 1.573 -1.539" robot_namespace="$(arg robot_namespace)">
+    <plugin_params>
+      <block>
+        <duration>0.3</duration>
+        <interval>0.3</interval>
+        <color>1 0.8</color>
+      </block>
+    </plugin_params>
+  </xacro:led>
+  <xacro:led led_prefix="right_lateral_rear" xyz="-0.066047 -0.212211 0.209188" rpy="0 1.573 -1.539" robot_namespace="$(arg robot_namespace)">
+    <plugin_params>
+      <block>
+        <duration>0.3</duration>
+        <interval>0.3</interval>
+        <color>1 0.8</color>
+      </block>
+    </plugin_params>
+  </xacro:led>
+  <xacro:led led_prefix="left_lateral_front" xyz="0.066047 0.212211 0.209188" rpy="0 1.573 1.539" robot_namespace="$(arg robot_namespace)">
+    <plugin_params>
+      <block>
+        <duration>0.3</duration>
+        <interval>0.3</interval>
+        <color>1 0.8</color>
+      </block>
+    </plugin_params>
+  </xacro:led>
+  <xacro:led led_prefix="left_lateral_rear" xyz="-0.066047 0.212211 0.209188" rpy="0 1.573 1.539" robot_namespace="$(arg robot_namespace)">
     <plugin_params>
       <block>
@@ -225,10 +225,11 @@
     </plugin>
   </gazebo>
+  <!--
   <gazebo>
     <plugin name="imu_controller" filename="libhector_gazebo_ros_imu.so">
       <robotNamespace>$(arg robot_namespace)</robotNamespace>
       <updateRate>50.0</updateRate>
-      <frameId>$(arg tfpre)base_link</frameId>
-      <bodyName>base_link</bodyName>
+      <frameId>$(arg robot_namespace)/base_link</frameId>
+      <bodyName>$(arg robot_namespace)/base_link</bodyName>
       <topicName>imu/data</topicName>
       <accelDrift>0.005 0.005 0.005</accelDrift>
@@ -244,6 +245,6 @@
       <robotNamespace>$(arg robot_namespace)</robotNamespace>
       <updateRate>40</updateRate>
-      <bodyName>base_link</bodyName>
-      <frameId>$(arg tfpre)base_link</frameId>
+      <bodyName>$(arg robot_namespace)/base_link</bodyName>
+      <frameId>$(arg robot_namespace)/base_link</frameId>
       <topicName>navsat/fix</topicName>
       <velocityTopicName>navsat/vel</velocityTopicName>
@@ -255,4 +256,5 @@
     </plugin>
   </gazebo>
+  -->
   <!-- Optional custom includes. -->
   <xacro:include filename="$(arg urdf_extras)" />

Commit message: More namespaces.
--HG--
branch : namespaces_for_rviz

File: x1_description/urdf/decorations.urdf.xacro (robot description, xacro)
@@ -24,12 +24,12 @@
   <xacro:macro name="x1_decorate" params="robot_namespace">
     <!-- Spawn X1 chassis -->
-    <link name="top_chassis_link">
+    <link name="${robot_namespace}/top_chassis_link">
     </link>
     <!-- Attach chassis to the robot -->
     <joint name="top_chassis_joint" type="fixed">
       <parent link="${robot_namespace}/base_link" />
-      <child link="top_chassis_link" />
+      <child link="${robot_namespace}/top_chassis_link" />
     </joint>
-    <link name="top_plate_link">
+    <link name="${robot_namespace}/top_plate_link">
       <visual>
         <origin xyz="0 0 0" rpy="0 0 0" />
@@ -54,21 +54,21 @@
     <joint name="top_plate_joint" type="fixed">
       <parent link="${robot_namespace}/base_link" />
-      <child link="top_plate_link"/>
+      <child link="${robot_namespace}/top_plate_link"/>
       <origin xyz="0.0812 0 0.245" rpy="0 0 0"/>
     </joint>
     <!-- Top plate front link -->
     <joint name="top_plate_front_joint" type="fixed">
-      <parent link="top_plate_link" />
-      <child link="top_plate_front_link"/>
+      <parent link="${robot_namespace}/top_plate_link" />
+      <child link="${robot_namespace}/top_plate_front_link"/>
       <origin xyz="0.36367 0 0.00639" rpy="0 0 0"/>
     </joint>
     <!-- Top plate rear link-->
     <joint name="top_plate_rear_joint" type="fixed">
-      <parent link="top_plate_link" />
-      <child link="top_plate_rear_link"/>
+      <parent link="${robot_namespace}/top_plate_link" />
+      <child link="${robot_namespace}/top_plate_rear_link"/>
       <origin xyz="-0.36633 0 0.00639" rpy="0 0 0"/>
     </joint>
-    <link name="top_plate_front_link"/>
-    <link name="top_plate_rear_link"/>
+    <link name="${robot_namespace}/top_plate_front_link"/>
+    <link name="${robot_namespace}/top_plate_rear_link"/>
   </xacro:macro>
 </robot>

File: x1_description/urdf/headlight.urdf.xacro (robot description, xacro)
@@ -2,5 +2,5 @@
 <robot xmlns:xacro="http://ros.org/wiki/xacro" name="headlight">
   <xacro:macro name="headlight" params="headlight_prefix xyz rpy robot_namespace">
-    <link name="${headlight_prefix}_headlight_link">
+    <link name="${robot_namespace}/${headlight_prefix}_headlight_link">
       <visual>
         <origin xyz="0 0 0" rpy="0 0 0" />
@@ -19,11 +19,11 @@
       </inertial>
     </link>
-    <joint name="${headlight_prefix}_headlight" type="fixed">
+    <joint name="${robot_namespace}/${headlight_prefix}_headlight" type="fixed">
       <parent link="${robot_namespace}/base_link"/>
-      <child link="${headlight_prefix}_headlight_link"/>
+      <child link="${robot_namespace}/${headlight_prefix}_headlight_link"/>
       <origin xyz="${xyz}" rpy="${rpy}"/>
     </joint>
     <gazebo>
-      <model name="${headlight_prefix}_headlight">
+      <model name="${robot_namespace}/${headlight_prefix}_headlight">
         <pose>${xyz} ${rpy}</pose>
         <link name="body">
@@ -89,7 +89,7 @@
     </gazebo>
     <gazebo>
-      <joint name="${headlight_prefix}_headlight" type="fixed">
+      <joint name="${robot_namespace}/${headlight_prefix}_headlight" type="fixed">
         <parent>${robot_namespace}/base_link</parent>
-        <child>${headlight_prefix}_headlight::body</child>
+        <child>${robot_namespace}/${headlight_prefix}_headlight::body</child>
       </joint>
     </gazebo>

File: x1_description/urdf/led.urdf.xacro (robot description, xacro)
@@ -2,5 +2,5 @@
 <robot xmlns:xacro="http://ros.org/wiki/xacro" name="led">
   <xacro:macro name="led" params="led_prefix xyz rpy **plugin_params robot_namespace">
-    <link name="${led_prefix}_led_link">
+    <link name="${robot_namespace}/${led_prefix}_led_link">
       <visual name="marker">
         <origin xyz="0 0 0" rpy="0 0 0" />
@@ -21,9 +21,9 @@
     <joint name="${led_prefix}_led" type="fixed">
       <parent link="${robot_namespace}/base_link"/>
-      <child link="${led_prefix}_led_link"/>
+      <child link="${robot_namespace}/${led_prefix}_led_link"/>
       <origin xyz="${xyz}" rpy="${rpy}"/>
     </joint>
     <gazebo>
-      <model name="${led_prefix}_led">
+      <model name="${robot_namespace}/${led_prefix}_led">
         <pose>${xyz} ${rpy}</pose>
         <link name="body">
@@ -86,5 +86,5 @@
       <joint name="${led_prefix}_led" type="fixed">
         <parent>${robot_namespace}/base_link</parent>
-        <child>${led_prefix}_led::body</child>
+        <child>${robot_namespace}/${led_prefix}_led::body</child>
       </joint>
     </gazebo>

File: x1_description/urdf/wheel.urdf.xacro (robot description, xacro)
@@ -23,5 +23,5 @@
 <robot xmlns:xacro="http://ros.org/wiki/xacro" name="x1_wheel">
 	<xacro:macro name="x1_wheel" params="wheel_prefix *joint_pose robot_namespace">
-		<link name="${wheel_prefix}_wheel_link">
+		<link name="${robot_namespace}/${wheel_prefix}_wheel_link">
 			<inertial>
 				<mass value="2.637" />
@@ -42,5 +42,5 @@
 			</collision>
 		</link>
-		<gazebo reference="${wheel_prefix}_wheel_link">
+		<gazebo reference="${robot_namespace}/${wheel_prefix}_wheel_link">
 			<mu1 value="1.0"/>
 			<mu2 value="1.0"/>
@@ -50,6 +50,6 @@
 		</gazebo>
 		<joint name="${wheel_prefix}_wheel" type="continuous">
-      <parent link="${robot_namespace}/base_link"/>
-			<child link="${wheel_prefix}_wheel_link"/>
+            <parent link="${robot_namespace}/base_link"/>
+			<child link="${robot_namespace}/${wheel_prefix}_wheel_link"/>
 			<xacro:insert_block name="joint_pose"/>
 			<axis xyz="0 1 0" rpy="0 0 0" />

File: x1_description/urdf/x1.urdf.xacro (robot description, xacro)
@@ -74,12 +74,12 @@
   </link>
   <!-- Base footprint is on the ground under the robot -->
-  <link name="base_footprint"/>
+  <link name="$(arg robot_namespace)/base_footprint"/>
   <joint name="base_footprint_joint" type="fixed">
     <origin xyz="0 0 ${wheel_vertical_offset - wheel_radius}" rpy="0 0 0" />
     <parent link="$(arg robot_namespace)/base_link" />
-    <child link="base_footprint" />
+    <child link="$(arg robot_namespace)/base_footprint" />
   </joint>
   <!-- Interial link stores the robot's inertial information -->
-  <link name="inertial_link">
+  <link name="$(arg robot_namespace)/inertial_link">
     <inertial>
       <mass value="46.034" />
@@ -91,15 +91,15 @@
     <origin xyz="0 0 0" rpy="0 0 0" />
     <parent link="$(arg robot_namespace)/base_link" />
-    <child link="inertial_link" />
+    <child link="$(arg robot_namespace)/inertial_link" />
   </joint>
   <!-- IMU Link is the standard mounting position for the UM6 IMU.-->
   <!-- Can be modified with environment variables in /etc/ros/setup.bash -->
-  <link name="imu_link"/>
+  <link name="$(arg robot_namespace)/imu_link"/>
   <joint name="imu_joint" type="fixed">
     <origin xyz="$(optenv X1_IMU_XYZ 0.19 0 0.149)" rpy="$(optenv X1_IMU_RPY 0 -1.5708 3.1416)" />
     <parent link="$(arg robot_namespace)/base_link" />
-    <child link="imu_link" />
+    <child link="$(arg robot_namespace)/imu_link" />
   </joint>
-  <gazebo reference="imu_link">
+  <gazebo reference="$(arg robot_namespace)/imu_link">
   </gazebo>
   <!-- X1 wheel macros -->
